File: Kicad/BertheVario213-Shema.kicad_sch (KiCad schematic)
At the start: 17 parts, among them CN1 Temperature and humidity inte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, P1 Power supply base, P3 Extended IO, P4 SPEAK, P5 10 k ohms, SW1 SW_DIP_x01

Commit message: pcb Kicad
Parts:
- removed BMP180_Press1: ~, BertheShema:BMP180, symbol BertheLibrary:BMP180
- removed BT1: Battery_Cell, BertheShema:batterie, symbol Device:Battery_Cell
- removed CN1: Temperature and humidity interface, BertheShema:4 trous standard, symbol Connector_Generic:Conn_01x04
- removed ESP32-2432S028_WROOM-32: -, Symbol:KiCad-Logo2_5mm_SilkScreen, symbol BertheLibrary:ESP32
- removed Lipo-1S-to-5V1: -, BertheShema:1S-to-5v, symbol BertheLibrary:Lipo-to-5v
- removed P1: Power supply base, BertheShema:4 trous standard, symbol Connector_Generic:Conn_01x04
- removed P3: Extended IO, BertheShema:4 trous standard, symbol Connector_Generic:Conn_01x04
- removed P4: SPEAK, BertheShema:2 trous standard, symbol Connector_Generic:Conn_01x02
- removed P5: 10 k ohms, BertheShema:potentiometre, symbol Device:R_Potentiometer
- removed SW1: SW_DIP_x01, BertheShema:2 trous standard, symbol Switch:SW_DIP_x01
- removed Usb-C-charger1: -, BertheShema:Usb-C-Charger, symbol BertheLibrary:Usb_c_charger
- added MS5611: ~, BertheShema:MS5611, symbol BertheLibrary:MS5611
- added U1: ~, BertheShema:ESP32-D0WDQ6, symbol BertheLibrary:ESP32-D0WDQ6-V3
Connections:
- net GNDREF: now also R1.2, S1.1, MS5611.3 (GND), U1.2 (Gnd), U1.9 (Gnd)
- net at GPS-NEO6M1.4 (VCC), QMC5883_Mag1.1 (VCC), R2.1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: now also MS5611.4 (VIN), U1.1 (3v3)
- net at QMC5883_Mag1.3 (SCL), R3.2: now also MS5611.2 (SCL), U1.22 (SCL)
- net at QMC5883_Mag1.4 (SDA), R2.2: now also MS5611.1 (SDA), U1.21 (SDA)
- net at GPS-NEO6M1.2 (TX): now also U1.3 (Txd)
Other:
- note added: "IO21 SDA"
- note removed: "GND"
- note removed: "GND to VBat -"
- note removed: "IO21"
- note removed: "IO27 SDA"
- note removed: "IO35 to VBat +"
- note removed: "Rx"
- note removed: "Tx"
- note removed: "VIN"
- note removed: "Vdd to Out Battery converter"
- note removed: "ou shunt suivant preference"
- moved on the sheet: GPS-NEO6M1, QMC5883_Mag1, R2, R3

Commit message: progession pcb
Parts:
- added Q1: S8050, Package_TO_SOT_THT:TO-92_Inline, symbol Transistor_BJT:2SC1815
- added R2, R6: 10k, Resistor_THT:R_Axial_DIN0207_L6.3mm_D2.5mm_P10.16mm_Horizontal, symbol Device:R_Small
- added R5: 10K, Resistor_THT:R_Axial_DIN0207_L6.3mm_D2.5mm_P10.16mm_Horizontal, symbol Device:R_Small
- added SW1: Gauche, BertheShema:switch, symbol Switch:SW_Push
- added SW2: Centre, BertheShema:switch, symbol Switch:SW_Push
- added SW3: Droit, BertheShema:switch, symbol Switch:SW_Push
- R1: value 3.6 ohms -> 1K
- renumbered R2 to R3, R3 to R4
Connections:
- net GNDREF: now also Q1.1 (E), R2.2, R6.2, SW1.2, SW2.2, SW3.2; no longer R1.2, S1.1
- net at R1.1: now also U1.34 (Speaker); no longer S1.2
- net at U1.6 (Vbat): now also S1.2, R5.1
- new net: R5.2, R6.1, U1.36 (VBat)
- new net: SW3.1, U1.13 (Bouton_Droit)
- new net: SW1.1, U1.14 (Bouton_Gauche)
- new net: SW2.1, U1.15 (Bouton_Centre)
- new net: Q1.2 (C), S1.1
- new net: Q1.3 (B), R1.2, R2.1

Commit message: progression pcb
Other:
- title: BertheVarioTac -> BertheVario213
Changed lines of the file:
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@@
   (paper "A4")
   (title_block
-    (title "BertheVarioTac")
+    (title "BertheVario213")
     (date "2025-02-15")
     (rev "1.0")

Commit message: doc concepteur
Parts:
- S1: value Speaker 2W 8ohms -> Speaker 1W 80 ohms
Changed lines of the file:
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@@
     (title "BertheVario213")
     (date "2025-02-15")
-    (rev "1.0")
+    (rev "1.01")
     (comment 1 "Author : SpinBerthe")
   )
@@
       (effects (font (size 1.27 1.27)) (justify left))
     )
-    (property "Value" "Speaker 2W 8ohms" (at 39.37 78.74 0)
-      (effects (font (size 1.27 1.27)) (justify left))
-    )
+    (property "Value" "Speaker 1W 80 ohms" (at 39.37 78.74 0)
+      (effects (font (size 1.27 1.27)) (justify left))
+    )
