File: Kicad/BertheVario213-Shema.kicad_sch (KiCad schematic)
At the start: 15 parts, among them Q1 S8050, SW1 Gauche, SW2 Centre, SW3 Droit

Commit message: son vbat
Connections:
- net at R1.1: now also U1.26 (Speaker); no longer U1.34 (Speaker)
Changed lines of the file:
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@@
     (title "BertheVario213")
     (date "2025-02-15")
-    (rev "1.02")
+    (rev "1.03")
     (comment 1 "Author : SpinBerthe")
   )
@@
     (pin "13")
     (pin "36")
-    (pin "34")
+    (pin "26")
     (instances
       (project "BertheVario213-Shema"

Commit message: son vbat
Connections:
- net at R1.1: now also U1.25 (Speaker); no longer U1.26 (Speaker)
Changed lines of the file:
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@@
     (title "BertheVario213")
     (date "2025-02-15")
-    (rev "1.03")
+    (rev "1.04")
     (comment 1 "Author : SpinBerthe")
   )
@@
     (pin "13")
     (pin "36")
-    (pin "26")
+    (pin "25")
     (instances
       (project "BertheVario213-Shema"

Commit message: mise a jour kicad
Connections:
- net at R5.1, U1.6 (Vbat): no longer S1.2
- new net: S1.2, U1.5 (5V)
Other:
- moved on the sheet: Q1, R2, R3, R5, R6, S1
