File: Kicad/BertheVario213-Shema.kicad_sch (KiCad schematic)
At the start: 15 parts, among them Q1 S8050, SW1 Gauche, SW2 Centre, SW3 Droit

Commit message: pcb
Connections:
- net at U1.5 (5V): no longer S1.2
- net at R5.1, U1.6 (Vbat): now also S1.2
Changed lines of the file:
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@@
     (title "BertheVario213")
     (date "2025-02-19")
-    (rev "1.06")
+    (rev "1.07")
     (comment 1 "Author : SpinBerthe")
   )
@@
   (junction (at 198.12 119.38) (diameter 0) (color 0 0 0 0)
   )
+  (junction (at 85.09 77.47) (diameter 0) (color 0 0 0 0)
+  )
   (junction (at 165.1 59.69) (diameter 0) (color 0 0 0 0)
   )
@@
     (stroke (width 0) (type default))
   )
-  (wire (pts (xy 80.01 91.44) (xy 142.24 91.44))
+  (wire (pts (xy 85.09 91.44) (xy 142.24 91.44))
     (stroke (width 0) (type default))
   )
@@
     (stroke (width 0) (type default))
   )
-  (wire (pts (xy 80.01 74.93) (xy 87.63 74.93))
-    (stroke (width 0) (type default))
-  )
   (wire (pts (xy 226.06 110.49) (xy 246.38 110.49))
     (stroke (width 0) (type default))
@@
     (stroke (width 0) (type default))
   )
-  (wire (pts (xy 80.01 74.93) (xy 80.01 91.44))
-    (stroke (width 0) (type default))
-  )
+  (wire (pts (xy 85.09 77.47) (xy 85.09 91.44))
+    (stroke (width 0) (type default))
+  )

Commit message: pcb pb
Parts:
- removed Q1: S8050, Package_TO_SOT_THT:TO-92_Inline, symbol Transistor_BJT:2SC1815
- removed SW1: Gauche, BertheShema:switch, symbol Switch:SW_Push
- removed SW2: Centre, BertheShema:switch, symbol Switch:SW_Push
- removed SW3: Droit, BertheShema:switch, symbol Switch:SW_Push
- added Q1: S8050, BertheShema:S8050, symbol BertheLibrary:S8050
- added SW1: bas, BertheShema:switch, symbol BertheLibrary:SW_DIP_x01
- added SW2: milieu, BertheShema:switch, symbol BertheLibrary:SW_DIP_x01
- added SW3: haut, BertheShema:switch, symbol BertheLibrary:SW_DIP_x01
- S1: value Speaker 1W 80 ohms -> Speaker 2W 8 ohms
Connections:
- net GNDREF: now also Q1.1 (E), SW1.2, SW2.2, SW3.2
- net at U1.13 (Bouton_Droit): now also SW3.1
- net at U1.14 (Bouton_Gauche): now also SW1.1
- net at U1.15 (Bouton_Centre): now also SW2.1
- net at S1.1: now also Q1.3 (C)
- net at R1.2, R2.1: now also Q1.2 (B)

Commit message: pcb a verifier
Parts:
- SW1: value bas -> gauche
- SW2: value milieu -> centre
- SW3: value haut -> droite
Changed lines of the file:
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@@
       (effects (font (size 1.27 1.27)))
     )
-    (property "Value" "milieu" (at 81.28 158.75 0)
+    (property "Value" "centre" (at 81.28 158.75 0)
       (effects (font (size 1.27 1.27)))
     )
@@
       (effects (font (size 1.27 1.27)))
     )
-    (property "Value" "bas" (at 55.88 158.75 0)
+    (property "Value" "gauche" (at 55.88 158.75 0)
       (effects (font (size 1.27 1.27)))
     )
@@
       (effects (font (size 1.27 1.27)))
     )
-    (property "Value" "haut" (at 104.14 158.75 0)
+    (property "Value" "droite" (at 104.14 158.75 0)
       (effects (font (size 1.27 1.27)))
     )

Commit message: pcb a verifier
Parts:
- R1, R2, R5, R6: footprint Resistor_THT:R_Axial_DIN0207_L6.3mm_D2.5mm_P10.16mm_Horizontal -> BertheShema:R_47
Connections:
- net at SW3.1: now also U1.26 (Bouton_Droit); no longer U1.13 (Bouton_Droit)
- net at SW1.1: now also U1.19 (Bouton_Gauche); no longer U1.14 (Bouton_Gauche)
- net at SW2.1: now also U1.32 (Bouton_Centre); no longer U1.15 (Bouton_Centre)
Changed lines of the file:
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@@
       (effects (font (size 1.27 1.27)) (justify left))
     )
-    (property "Footprint" "Resistor_THT:R_Axial_DIN0207_L6.3mm_D2.5mm_P10.16mm_Horizontal" (at 144.78 44.45 0)
+    (property "Footprint" "BertheShema:R_47" (at 144.78 44.45 0)
       (effects (font (size 1.27 1.27)) hide)
     )
@@
     (pin "6")
     (pin "4")
-    (pin "14")
-    (pin "15")
-    (pin "13")
+    (pin "32")
+    (pin "26")
+    (pin "19")
     (pin "36")
     (pin "25")
@@
       (effects (font (size 1.27 1.27) italic) (justify left) hide)
     )
-    (property "Datasheet" "http://www.onsemi.com/pub_link/Collateral/2N2219-D.PDF" (at 175.26 59.69 0)
+    (property "Datasheet" "" (at 175.26 59.69 0)
       (effects (font (size 1.27 1.27)) (justify left) hide)
     )
@@
       (effects (font (size 1.27 1.27)) (justify left))
     )
-    (property "Footprint" "Resistor_THT:R_Axial_DIN0207_L6.3mm_D2.5mm_P10.16mm_Horizontal" (at 144.78 31.75 0)
+    (property "Footprint" "BertheShema:R_47" (at 144.78 31.75 0)
       (effects (font (size 1.27 1.27)) hide)
     )
@@
       (effects (font (size 1.27 1.27)))
     )
-    (property "Footprint" "Resistor_THT:R_Axial_DIN0207_L6.3mm_D2.5mm_P10.16mm_Horizontal" (at 161.29 59.69 0)
+    (property "Footprint" "BertheShema:R_47" (at 161.29 59.69 0)
       (effects (font (size 1.27 1.27)) hide)
     )
@@
       (effects (font (size 1.27 1.27)) (justify left))
     )
-    (property "Footprint" "Resistor_THT:R_Axial_DIN0207_L6.3mm_D2.5mm_P10.16mm_Horizontal" (at 165.1 64.77 0)
-      (effects (font (size 1.27 1.27)) hide)
-    )
+    (property "Footprint" "BertheShema:R_47" (at 165.1 64.77 0)
+      (effects (font (size 1.27 1.27)) hide)
+    )

Commit message: gps pb
Connections:
- net GNDREF: no longer U1.9 (Gnd)
- net at U1.3 (Txd): no longer GPS-NEO6M1.2 (TX)
- net at U1.4 (Rxd): now also GPS-NEO6M1.2 (TX)
Changed lines of the file:
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@@
   (title_block
     (title "BertheVario213")
-    (date "2025-02-21")
-    (rev "1.08")
+    (date "2025-02-22")
+    (rev "1.09")
     (comment 1 "Author : SpinBerthe")
   )
@@
     (stroke (width 0) (type default))
   )
-  (wire (pts (xy 125.73 71.12) (xy 125.73 82.55))
-    (stroke (width 0) (type default))
-  )
   (wire (pts (xy 85.09 91.44) (xy 142.24 91.44))
     (stroke (width 0) (type default))
@@
     (stroke (width 0) (type default))
   )
-  (wire (pts (xy 118.11 71.12) (xy 125.73 71.12))
-    (stroke (width 0) (type default))
-  )
   (wire (pts (xy 226.06 110.49) (xy 246.38 110.49))
     (stroke (width 0) (type default))
@@
     (stroke (width 0) (type default))
   )
-  (wire (pts (xy 74.93 54.61) (xy 87.63 54.61))
+  (wire (pts (xy 74.93 57.15) (xy 87.63 57.15))
     (stroke (width 0) (type default))
   )
@@
     (stroke (width 0) (type default))
   )
-  (wire (pts (xy 74.93 54.61) (xy 74.93 140.97))
+  (wire (pts (xy 74.93 57.15) (xy 74.93 140.97))
     (stroke (width 0) (type default))
   )
@@
     (pin "3")
     (pin "2")
-    (pin "9")
     (pin "22")
     (pin "1")
@@
         )
       )
-    )
-  )
-  (symbol (lib_id "power:GNDREF") (at 125.73 82.55 0) (unit 1)
-    (in_bom yes) (on_board yes) (dnp no) (fields_autoplaced)
-    (property "Reference" "#PWR03" (at 125.73 88.9 0)
-      (effects (font (size 1.27 1.27)) hide)
-    )
-    (property "Value" "GNDREF" (at 125.73 87.63 0)
-      (effects (font (size 1.27 1.27)))
-    )
-    (property "Footprint" "" (at 125.73 82.55 0)
-      (effects (font (size 1.27 1.27)) hide)
-    )
-    (property "Datasheet" "" (at 125.73 82.55 0)
-      (effects (font (size 1.27 1.27)) hide)
-    )
-    (pin "1")
-    (instances
-      (project "BertheVario213-Shema"
-        (path "/20a72893-107a-4d28-9717-d104a5df1eab"
-          (reference "#PWR03") (unit 1)
-        )
-      )

Commit message: modif pcb
Parts:
- added jumper1: ~, BertheShema:jumper, symbol BertheLibrary:jumper
Connections:
- net at U1.4 (Rxd): now also jumper1.1; no longer GPS-NEO6M1.2 (TX)
- new net: GPS-NEO6M1.2 (TX), jumper1.2
Changed lines of the file:
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@@
   (title_block
     (title "BertheVario213")
-    (date "2025-02-22")
-    (rev "1.09")
+    (date "2025-02-23")
+    (rev "1.10")
     (comment 1 "Author : SpinBerthe")
   )
@@
     (stroke (width 0) (type default))
   )
+  (wire (pts (xy 144.78 140.97) (xy 246.38 140.97))
+    (stroke (width 0) (type default))
+  )
   (wire (pts (xy 120.65 170.18) (xy 111.76 170.18))
     (stroke (width 0) (type default))
@@
     (stroke (width 0) (type default))
   )
-  (wire (pts (xy 74.93 140.97) (xy 246.38 140.97))
+  (wire (pts (xy 74.93 140.97) (xy 134.62 140.97))
     (stroke (width 0) (type default))
   )
@@
         )
       )
+    )
+  )
+  (symbol (lib_id "BertheLibrary:jumper") (at 139.7 140.97 0) (unit 1)
+    (in_bom yes) (on_board yes) (dnp no) (fields_autoplaced)
+    (property "Reference" "jumper1" (at 139.7 137.16 0)
+      (effects (font (size 1.27 1.27)))
+    )
+    (property "Value" "~" (at 139.7 140.97 0)
+      (effects (font (size 1.27 1.27)))
+    )
+    (property "Footprint" "BertheShema:jumper" (at 139.7 140.97 0)
+      (effects (font (size 1.27 1.27)) hide)
+    )
+    (property "Datasheet" "" (at 139.7 140.97 0)
+      (effects (font (size 1.27 1.27)) hide)
+    )
+    (pin "2")
+    (pin "1")
+    (instances
+      (project "BertheVario213-Shema"
+        (path "/20a72893-107a-4d28-9717-d104a5df1eab"
+          (reference "jumper1") (unit 1)
+        )
+      )

Commit message: pcb ok a verifier
Connections:
- net GNDREF: now also U1.41 (Gnd); no longer U1.2 (Gnd)
- net at GPS-NEO6M1.4 (VCC), MS5611.4 (VIN), QMC5883_Mag1.1 (VCC)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: now also U1.40 (3v3); no longer U1.1 (3v3)
- net at jumper1.1: now also U1.43 (Rxd); no longer U1.4 (Rxd)
- net at R5.1, S1.2: now also U1.45 (Vbat); no longer U1.6 (Vbat)
Changed lines of the file:
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@@
   (title_block
     (title "BertheVario213")
-    (date "2025-02-23")
-    (rev "1.10")
+    (date "2025-02-24")
+    (rev "1.12")
     (comment 1 "Author : SpinBerthe")
   )
@@
     )
     (pin "21")
-    (pin "3")
-    (pin "2")
+    (pin "41")
+    (pin "43")
     (pin "22")
-    (pin "1")
-    (pin "6")
-    (pin "4")
+    (pin "45")
+    (pin "40")
     (pin "32")
     (pin "26")
@@
     (pin "36")
     (pin "25")
-    (pin "5")
     (instances
       (project "BertheVario213-Shema"
