File: Kicad/BertheVario213-Shema.kicad_pcb (KiCad board)
At the start: 2 copper layers, 0 parts

Commit message: pcb Kicad
Parts:
- added GPS-NEO6M1: -, BertheShema:GPSNEO6V2, F.Cu at (139.8, 101.0)
- added MS5611: ~, BertheShema:MS5611, F.Cu at (155.5, 51.4)
- added QMC5883_Mag1: ~, BertheShema:QMC5883, F.Cu at (163.6, 104.0)
- added R1: 3.6 ohms, Resistor_THT:R_Axial_DIN0207_L6.3mm_D2.5mm_P10.16mm_Horizontal, F.Cu at (104.5, 63.0)
- added R2: 4.7k, BertheShema:R_47, F.Cu at (109.5, 66.5)
- added R3: 4.7k, BertheShema:R_47, F.Cu at (109.5, 69.5)
- added S1: Speaker 2W 8ohms, BertheShema:2 trous standard, F.Cu at (104.3, 74.9)
- added U1: ~, BertheShema:ESP32-D0WDQ6, F.Cu at (148.8, 49.3)

Commit message: empreintes Kicad
Parts:
- moved R1 88.4 mm to (183.5, 23.5), turned to -90 degrees
- moved S1 84.8 mm to (171.6, 23.3), turned to -90 degrees
- moved R2 80.1 mm to (180.0, 28.5), turned to -90 degrees
- moved R3 79.0 mm to (177.0, 28.5), turned to -90 degrees
- moved GPS-NEO6M1 31.9 mm to (165.0, 81.5)
- moved QMC5883_Mag1 30.5 mm to (171.5, 133.5)
- moved MS5611 7.04 mm to (148.8, 49.5), turned to -90 degrees

Commit message: progession pcb
Parts:
- added Q1: S8050, Package_TO_SOT_THT:TO-92_Inline, F.Cu at (141.2, 117.3)
- added R1: 1K, Resistor_THT:R_Axial_DIN0207_L6.3mm_D2.5mm_P10.16mm_Horizontal, F.Cu at (140.8, 99.8)
- added R2: 10k, Resistor_THT:R_Axial_DIN0207_L6.3mm_D2.5mm_P10.16mm_Horizontal, F.Cu at (140.8, 103.9)
- added R5: 10K, Resistor_THT:R_Axial_DIN0207_L6.3mm_D2.5mm_P10.16mm_Horizontal, F.Cu at (140.8, 108.0)
- added R6: 10k, Resistor_THT:R_Axial_DIN0207_L6.3mm_D2.5mm_P10.16mm_Horizontal, F.Cu at (140.8, 112.0)
- added SW1: Gauche, BertheShema:switch, F.Cu at (135.5, 100.4)
- added SW2: Centre, BertheShema:switch, F.Cu at (135.5, 108.0)
- added SW3: Droit, BertheShema:switch, F.Cu at (135.5, 115.6)
- moved R1 37.9 mm to (146.5, 31.5), turned to 0 degrees
- moved S1 32.3 mm to (146.3, 43.4), turned to 0 degrees
- moved R3 29.2 mm to (151.5, 35.0), turned to 0 degrees
- moved R4 27.2 mm to (151.5, 38.0), turned to 0 degrees
- moved MS5611 5.27 mm to (147.1, 54.5)
- renumbered R2 to R3, R3 to R4
Connections:
- S1 pad 1: GNDREF -> Net-(Q1-C)
- S1 pad 2: Net-(R1-Pad1) -> Net-(U1-Vbat)
- U1 pad 13: (no net) -> Net-(U1-Bouton_Droit)
- U1 pad 14: (no net) -> Net-(U1-Bouton_Gauche)
- U1 pad 15: (no net) -> Net-(U1-Bouton_Centre)
- U1 pad 34: (no net) -> Net-(U1-Speaker)
- U1 pad 36: (no net) -> Net-(U1-VBat)
- U1 pad 6: unconnected-(U1-Vbat-Pad6) -> Net-(U1-Vbat)
Other:
- board outline added: 49 x 135 mm

Commit message: modif pcb
Parts:
- removed the R1 at (146.5, 31.5)
- S1: value Speaker 2W 8ohms -> Speaker 1W 80 ohms
- moved R3 59.1 mm to (149.0, 94.0), turned to -90 degrees
- moved R4 56.1 mm to (154.0, 94.0), turned to -90 degrees
- moved SW3 53.6 mm to (132.5, 62.1)
- moved GPS-NEO6M1 49.9 mm to (157.0, 130.8), turned to 90 degrees
- moved SW2 46.4 mm to (142.5, 62.1)
- moved Q1 44.3 mm to (150.7, 74.0)
- moved MS5611 43.4 mm to (138.0, 96.9), turned to 0 degrees
- moved SW1 42.2 mm to (153.5, 62.3)
- moved U1 40.9 mm to (140.3, 89.3)
- moved QMC5883_Mag1 30.2 mm to (157.1, 160.0)
- moved R2 30.0 mm to (132.9, 75.0)
- moved R5 30.0 mm to (132.9, 79.0)
- moved R6 30.0 mm to (132.9, 83.0)
- moved R1 30.0 mm to (132.9, 70.9)
- moved S1 12.6 mm to (145.0, 56.0), turned to 90 degrees
Connections:
- S1 pad 2: Net-(U1-Vbat) -> Net-(U1-5V)
- U1 pad 25: (no net) -> Net-(U1-Speaker)
- U1 pad 34: Net-(U1-Speaker) -> (no net)
- U1 pad 5: (no net) -> Net-(U1-5V)
Other:
- board size 49 x 135 mm -> 43 x 122 mm

Commit message: modif pcb
Parts:
- moved GPS-NEO6M1 31.1 mm to (125.9, 129.8), turned to -90 degrees
- moved S1 22.2 mm to (163.0, 69.0), turned to 0 degrees
- moved R4 9.00 mm to (154.0, 85.0)
- moved QMC5883_Mag1 8.05 mm to (158.0, 152.0)
- moved MS5611 4.81 mm to (133.2, 96.9)
- moved SW3 1.07 mm to (132.0, 63.0)
- moved R3 1.00 mm to (150.0, 94.0)
- moved SW2 0.92 mm to (142.5, 63.0)
- moved SW1 0.73 mm to (153.5, 63.0)
Other:
- board size 43 x 122 mm -> 42.5 x 109 mm

Commit message: modif pcb
Parts:
- moved S1 64.5 mm to (163.0, 133.5)
- moved QMC5883_Mag1 1.10 mm to (157.5, 153.0)
Routing:
- net GNDREF: track 0.00 -> 244.0 mm
- net Net-(GPS-NEO6M1-VCC): track 0.00 -> 144.1 mm, vias 0 -> 1
- net Net-(MS5611-SDA): track 0.00 -> 137.7 mm, vias 0 -> 2
- net Net-(MS5611-SCL): track 0.00 -> 110.2 mm
- net Net-(Q1-C): track 0.00 -> 85.8 mm, vias 0 -> 2
- net Net-(U1-5V): track 0.00 -> 56.4 mm
- net Net-(U1-Bouton_Gauche): track 0.00 -> 49.9 mm, vias 0 -> 2
- net Net-(U1-Bouton_Centre): track 0.00 -> 46.7 mm
- net Net-(U1-Speaker): track 0.00 -> 34.3 mm
- net Net-(U1-In_Vbat): track 0.00 -> 29.6 mm, vias 0 -> 1
- net Net-(U1-Vbat): track 0.00 -> 28.8 mm
- net Net-(Q1-B): track 0.00 -> 26.2 mm

Commit message: modif pcb
Parts:
- moved SW3 37.5 mm to (167.2, 76.0), turned to -90 degrees
- moved SW1 37.1 mm to (167.2, 97.5), turned to -90 degrees
- moved SW2 34.1 mm to (167.2, 86.5), turned to -90 degrees
- moved R4 4.03 mm to (153.5, 81.0)
- moved Q1 3.07 mm to (147.7, 73.4)
- moved S1 1.15 mm to (162.5, 132.5), turned to -90 degrees
- moved GPS-NEO6M1 0.71 mm to (126.4, 129.3)
Routing:
- net Net-(Q1-C): track 85.8 -> 0.00 mm, vias 2 -> 0
- net Net-(U1-Bouton_Gauche): track 49.9 -> 0.00 mm, vias 2 -> 0
- net Net-(U1-Bouton_Centre): track 46.7 -> 0.00 mm
- net Net-(MS5611-SDA): track 137.7 -> 107.4 mm, vias 2 -> 3
- net GNDREF: track 244.0 -> 219.0 mm, vias 0 -> 1
- net Net-(Q1-B): track 26.2 -> 21.0 mm
- net Net-(GPS-NEO6M1-VCC): track 144.1 -> 148.1 mm, vias 1 -> 4
- net Net-(U1-In_Vbat): track 29.6 -> 33.0 mm, vias 1 -> 0
- net Net-(MS5611-SCL): track 110.2 -> 111.2 mm
- net Net-(U1-Speaker): track 34.3 -> 34.9 mm
Other:
- board size 42.5 x 109 mm -> 48 x 95 mm

Commit message: pcb
Parts:
- moved Q1 2.96 mm to (148.5, 70.5), turned to -90 degrees
- moved MS5611 2.06 mm to (135.2, 96.4)
- moved R4 1.87 mm to (154.5, 79.4)
- moved R3 1.80 mm to (151.5, 93.0)
Routing:
- net Net-(GPS-NEO6M1-TX): track 0.00 -> 93.2 mm, vias 0 -> 1
- net Net-(Q1-C): track 0.00 -> 75.7 mm
- net Net-(MS5611-SCL): track 111.2 -> 130.3 mm, vias 0 -> 1
- net Net-(U1-Speaker): track 34.9 -> 41.7 mm, vias 0 -> 2
- net GNDREF: track 219.0 -> 213.1 mm
- net Net-(Q1-B): track 21.0 -> 25.4 mm
- net Net-(U1-In_Vbat): track 33.0 -> 28.9 mm
- net Net-(GPS-NEO6M1-VCC): track 148.1 -> 147.6 mm, vias 4 -> 1
- net Net-(MS5611-SDA): track 107.4 -> 107.8 mm, vias 3 -> 2
- net Net-(U1-Vbat): vias 0 -> 1
Other:
- board size 48 x 95 mm -> 48 x 94.5 mm
