File: Kicad/BertheVario213-Shema.kicad_pcb (KiCad board)
At the start: 2 copper layers, 42 x 101.5 mm, 15 parts, among them Q1 S8050, SW1 gauche, SW2 centre, SW3 droite

Commit message: modif pcb
Parts:
- moved S1 10.2 mm to (151.0, 138.0), turned to -90 degrees
- moved GPS-NEO6M1 10.0 mm to (135.3, 125.9), turned to 180 degrees
- moved QMC5883_Mag1 2.50 mm to (155.0, 148.5)
Routing:
- net Net-(U1-Bouton_Droit): track 116.9 -> 49.3 mm, vias 1 -> 0
- net Net-(GPS-NEO6M1-VCC): track 150.2 -> 120.4 mm
- net Net-(Q1-C): track 82.6 -> 66.5 mm, vias 1 -> 0
- net Net-(U1-Vbat): track 88.8 -> 100.9 mm, vias 0 -> 1
- net Net-(MS5611-SDA): track 100.3 -> 108.2 mm
- net GNDREF: track 206.4 -> 213.9 mm
- net Net-(U1-Bouton_Gauche): track 50.0 -> 42.8 mm, vias 2 -> 1
- net Net-(Q1-B): track 24.6 -> 19.2 mm
- net Net-(GPS-NEO6M1-TX): track 50.3 -> 45.2 mm
- net Net-(U1-Bouton_Centre): track 32.4 -> 36.9 mm
- net Net-(U1-In_Vbat): track 36.1 -> 32.5 mm, vias 1 -> 0
- net Net-(U1-Speaker): track 31.7 -> 33.3 mm, vias 1 -> 0
Other:
- board size 42 x 101.5 mm -> 42 x 96.5 mm

Commit message: gps pb
Parts:
- moved QMC5883_Mag1 2.06 mm to (157.0, 148.0)
Connections:
- U1 pad 3: Net-(GPS-NEO6M1-TX) -> unconnected-(U1-Txd-Pad3)
- U1 pad 4: unconnected-(U1-Rxd-Pad4) -> Net-(GPS-NEO6M1-TX)
Routing:
- net Net-(GPS-NEO6M1-VCC): track 120.4 -> 153.0 mm, vias 0 -> 1
- net Net-(U1-Vbat): track 100.9 -> 79.3 mm, vias 1 -> 0
- net Net-(Q1-C): track 66.5 -> 85.9 mm, vias 0 -> 2
- net Net-(MS5611-SDA): track 108.2 -> 91.3 mm, vias 2 -> 0
- net Net-(MS5611-SCL): track 107.8 -> 120.1 mm, vias 0 -> 1
- net Net-(U1-Speaker): track 33.3 -> 43.6 mm, vias 0 -> 1
- net GNDREF: track 213.9 -> 204.3 mm
- net Net-(U1-Bouton_Droit): track 49.3 -> 42.0 mm
- net Net-(U1-In_Vbat): track 32.5 -> 39.8 mm
- net Net-(U1-Bouton_Gauche): track 42.8 -> 49.7 mm
- net Net-(U1-Bouton_Centre): track 36.9 -> 31.7 mm

Commit message: modif pcb
Parts:
- added jumper1: ~, BertheShema:jumper, F.Cu at (155.0, 121.0)
- moved MS5611 1.98 mm to (143.8, 90.8)
- moved Q1 1.98 mm to (147.0, 74.3)
- moved R1 1.98 mm to (134.9, 71.2)
- moved R2 1.98 mm to (134.9, 75.2)
- moved R3 1.98 mm to (152.8, 92.5)
- moved R4 1.98 mm to (152.8, 76.8)
- moved R5 1.98 mm to (134.9, 79.3)
- moved R6 1.98 mm to (134.9, 83.3)
- moved U1 1.98 mm to (139.2, 89.8)
- moved QMC5883_Mag1 1.00 mm to (156.0, 148.0)
Connections:
- U1 pad 4: Net-(GPS-NEO6M1-TX) -> Net-(U1-Rxd)
Routing:
- net Net-(U1-Bouton_Gauche): track 49.7 -> 129.7 mm, vias 1 -> 2
- net Net-(U1-Rxd): track 0.00 -> 55.3 mm, vias 0 -> 2
- net Net-(GPS-NEO6M1-VCC): track 153.0 -> 120.9 mm, vias 1 -> 0
- net Net-(GPS-NEO6M1-TX): track 45.5 -> 19.8 mm
- net GNDREF: track 204.3 -> 225.7 mm
- net Net-(Q1-C): track 85.9 -> 67.5 mm
- net Net-(MS5611-SDA): track 91.3 -> 106.0 mm, vias 0 -> 1
- net Net-(MS5611-SCL): track 120.1 -> 112.3 mm
- net Net-(U1-Bouton_Centre): track 31.7 -> 24.5 mm
- net Net-(U1-Vbat): track 79.3 -> 85.0 mm
- net Net-(U1-Bouton_Droit): track 42.0 -> 37.2 mm, vias 0 -> 1
- net Net-(U1-In_Vbat): track 39.8 -> 41.6 mm, vias 0 -> 1
- net Net-(U1-Speaker): track 43.6 -> 44.0 mm, vias 1 -> 0
Other:
- outline, holes or cut-outs redrawn

Commit message: pcb ok a verifier
Connections:
- U1 pad 2: GNDREF -> (no net)
- U1 pad 40: (no net) -> Net-(GPS-NEO6M1-VCC)
- U1 pad 41: (no net) -> GNDREF
Routing:
- net Net-(U1-Bouton_Gauche): track 129.7 -> 45.2 mm, vias 2 -> 0
- net GNDREF: track 225.7 -> 196.5 mm
- net Net-(U1-Bouton_Droit): track 37.2 -> 53.8 mm
- net Net-(U1-Speaker): track 44.0 -> 29.4 mm
- net Net-(U1-In_Vbat): track 41.6 -> 33.0 mm
- net Net-(MS5611-SDA): track 106.0 -> 111.7 mm, vias 1 -> 3
- net Net-(U1-Bouton_Centre): track 24.5 -> 29.7 mm
- net Net-(U1-Vbat): track 85.0 -> 81.3 mm
- net Net-(Q1-C): track 67.5 -> 69.3 mm, vias 2 -> 1
- net Net-(GPS-NEO6M1-VCC): track 120.9 -> 122.5 mm, vias 0 -> 1
- net Net-(MS5611-SCL): track 112.3 -> 113.2 mm, vias 1 -> 0
- net Net-(U1-Rxd): track 55.3 -> 54.8 mm, vias 2 -> 1
- added copper zone on B.Cu, net GNDREF
- added copper zone on F.Cu, net GNDREF

Commit message: modif pcb
Parts:
- moved R3 28.1 mm to (147.1, 120.0), turned to 180 degrees
- moved R1 19.7 mm to (154.0, 76.0), turned to -90 degrees
- moved jumper1 13.3 mm to (158.0, 134.0), turned to -90 degrees
- moved R4 11.8 mm to (151.5, 88.5)
- moved MS5611 11.1 mm to (135.0, 97.5), turned to 0 degrees
- moved R6 5.38 mm to (135.5, 78.0)
- moved R5 4.24 mm to (135.5, 83.5), turned to 180 degrees
- moved R2 3.30 mm to (135.5, 72.0)
- moved SW3 1.55 mm to (132.8, 64.8)
- moved SW1 1.45 mm to (155.8, 64.8)
- moved Q1 0.84 mm to (147.2, 75.1)
Routing:
- net GNDREF: track 196.5 -> 0.00 mm
- net Net-(U1-Rxd): track 54.8 -> 114.2 mm
- net Net-(MS5611-SDA): track 111.7 -> 82.2 mm, vias 3 -> 0
- net Net-(GPS-NEO6M1-VCC): track 122.5 -> 151.4 mm, vias 1 -> 0
- net Net-(GPS-NEO6M1-TX): track 19.8 -> 29.3 mm
- net Net-(U1-Vbat): track 81.3 -> 73.1 mm, vias 0 -> 1
- net Net-(U1-In_Vbat): track 33.0 -> 25.6 mm, vias 1 -> 0
- net Net-(U1-Bouton_Centre): track 29.7 -> 36.4 mm
- net Net-(MS5611-SCL): track 113.2 -> 106.7 mm
- net Net-(U1-Speaker): track 29.4 -> 24.5 mm
- net Net-(Q1-C): track 69.3 -> 73.5 mm
- net Net-(U1-Bouton_Gauche): track 45.2 -> 49.1 mm, vias 0 -> 1
- net Net-(U1-Bouton_Droit): track 53.8 -> 57.5 mm, vias 1 -> 0
- net Net-(Q1-B): track 19.2 -> 16.4 mm

Commit message: modif pcb
Routing:
- net Net-(U1-Rxd): track 114.2 -> 69.0 mm
- net Net-(GPS-NEO6M1-VCC): track 151.4 -> 131.6 mm, vias 0 -> 1
- net Net-(MS5611-SDA): track 82.2 -> 98.7 mm, vias 0 -> 1
- net Net-(U1-Speaker): track 24.5 -> 12.5 mm
- net Net-(U1-Bouton_Droit): track 57.5 -> 48.2 mm
- net Net-(Q1-C): track 73.5 -> 80.0 mm
- net Net-(U1-Vbat): track 73.1 -> 78.5 mm, vias 1 -> 2
- net Net-(U1-Bouton_Gauche): track 49.1 -> 52.6 mm, vias 1 -> 0
- net Net-(U1-In_Vbat): track 25.6 -> 23.9 mm
- net Net-(MS5611-SCL): track 106.7 -> 107.3 mm, vias 0 -> 1
